File: EagleFiles/LoRaWAN_FW_RevB.brd (EAGLE design)
At the start: 50.8 x 26.7 mm, 14 parts

Commit message: Updated Eagle files
Parts:
- removed C3: 470nF, adafruit:C0603
- added C1: 1uF, adafruit:C0603
- C2: value 1uF -> 470nF
- moved C2 11.6 mm to (22.9, 5.71)
Connections:
- net 3V: now also C1.1; no longer C3.1
- net GND: now also C1.2; no longer C3.2
Changed lines of the file:
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@@
 </autorouter>
 <elements>
-<element name="C3" library="adafruit" package="C0603" value="470nF" x="22.86" y="5.715" smashed="yes" rot="MR180"/>
+<element name="C2" library="adafruit" package="C0603" value="470nF" x="22.86" y="5.715" smashed="yes" rot="MR180"/>
 <element name="U$1" library="SparkFun-Aesthetics" package="OSHW-LOGO-M" value="" x="41.5925" y="1.27"/>
 <element name="LED2" library="adafruit" package="CHIPLED_0805" value="GREEN" x="3.81" y="5.87375" smashed="yes" rot="R90"/>
@@
 <element name="H1" library="holes" package="2,8-PAD" value="MOUNT-PAD-ROUND2.8" x="2.2225" y="20.6375"/>
 <element name="H2" library="holes" package="2,8-PAD" value="MOUNT-PAD-ROUND2.8" x="2.2225" y="2.2225"/>
-<element name="C2" library="adafruit" package="C0603" value="1uF" x="22.86" y="17.30375" smashed="yes" rot="MR180"/>
+<element name="C1" library="adafruit" package="C0603" value="1uF" x="22.86" y="17.30375" smashed="yes" rot="MR180"/>
 <element name="X1" library="adafruit" package="SMA_EDGELAUNCH" value="" x="0" y="11.43" smashed="yes">
 <attribute name="VALUE" x="5.08" y="3.81" size="0.8128" layer="27" ratio="10" rot="R180"/>
@@
 <contactref element="H1" pad="B2,8"/>
 <contactref element="LED1" pad="C"/>
+<contactref element="C1" pad="2"/>
 <contactref element="C2" pad="2"/>
-<contactref element="C3" pad="2"/>
 <contactref element="X1" pad="GND@4"/>
 <contactref element="X1" pad="GND@2"/>
@@
 <signal name="3V">
 <contactref element="R1" pad="2"/>
+<contactref element="C1" pad="1"/>
 <contactref element="C2" pad="1"/>
-<contactref element="C3" pad="1"/>
 <contactref element="U1" pad="12"/>
 <contactref element="U1" pad="34"/>
